File: E80-1800-pcb-universal/E80-1800-pcb-universal.kicad_pcb (KiCad board)
At the start: 2 copper layers, 382 x 159.6 mm, 321 parts, among them J1 SPI, J2 OLED, J3 USB_C_Receptacle_USB2.0, Q1 AO3400A, SW1 RST, SW2 BOOT, U1 SRV05-4, U2 XC6206P332MR, U3 STM32F072RBTx

Commit message: continued routing
Parts:
- moved C12 174.1 mm to (268.5, -8.45), turned to 90 degrees
- moved SW1 63.3 mm to (71.6, 110.6), turned to 0 degrees
- moved SW2 56.3 mm to (71.6, 118.0), turned to 0 degrees
- moved R11 9.45 mm to (261.9, -11.9)
- moved R9 3.82 mm to (263.6, -8.45)
- moved R10 3.81 mm to (265.2, -8.45), turned to 90 degrees
- moved C15 3.53 mm to (265.2, -11.9), turned to 270 degrees
- moved R12 3.53 mm to (263.6, -11.9), turned to 270 degrees
- moved C14 1.55 mm to (266.9, -8.45)
Connections:
- J2 pad 3: I2C_SCK -> I2C_SCL
- U3 pad 29: Net-(U3-Pad29) -> I2C_SCL
- U3 pad 30: Net-(U3-Pad30) -> I2C_SDA
- U3 pad 8: /sense_charge -> /sense_battV
- U3 pad 9: /sense_battV -> /sense_charge
Routing:
- net /BOOT: track 12.0 -> 368.8 mm, vias 1 -> 4
- net +3V3: track 121.1 -> 472.8 mm, vias 5 -> 7
- net /RST: track 2.89 -> 338.0 mm
- net I2C_SDA: track 0.00 -> 37.5 mm, vias 0 -> 1
- net I2C_SCL: track 0.00 -> 31.5 mm, vias 0 -> 1
- net +5V: track 2636.7 -> 2647.0 mm
- net GND: track 17.4 -> 7.39 mm, vias 34 -> 102
- net /sense_battV: track 15.3 -> 9.44 mm
- net COL14: track 193.9 -> 189.7 mm, vias 1 -> 3
- net /sense_charge: track 10.1 -> 12.4 mm, vias 1 -> 0
- net chgsense: track 0.00 -> 2.11 mm, vias 0 -> 1
- net ROW00: track 346.1 -> 347.5 mm
- net SPI_MOSI: track 10.7 -> 12.0 mm
- net SPI_MISO: track 11.7 -> 12.7 mm
- net SPI_SCK: track 12.2 -> 13.1 mm
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Other:
- board size 382 x 159.6 mm -> 382 x 160 mm

Commit message: finished pcb layout, added silk labels
Parts:
- added J4: Conn_01x05, Connector_JST:JST_SH_SM05B-SRSS-TB_1x05-1MP_P1.00mm_Horizontal, B.Cu at (294.2, -22.0)
- added JP1: BATT, Jumper:SolderJumper-2_P1.3mm_Bridged2Bar_Pad1.0x1.5mm, B.Cu at (295.7, -16.0)
- added R1: 4k7, Resistor_SMD:R_0603_1608Metric_Pad1.05x0.95mm_HandSolder, B.Cu at (260.9, -21.0)
- added R2: 4k7, Resistor_SMD:R_0603_1608Metric_Pad1.05x0.95mm_HandSolder, B.Cu at (260.9, -18.5)
- moved J1 5.67 mm to (283.3, -22.0), turned to 0 degrees
- moved SW1 0.20 mm to (71.4, 110.6)
- moved SW2 0.20 mm to (71.4, 118.0)
- renumbered R8 to R10, R9 to R11, R10 to R12, R11 to R13, R12 to R14, R1 to R3, R2 to R4, R3 to R5, R4 to R6, R5 to R7, R6 to R8, R7 to R9
Connections:
- F1 pad 1: +5V -> VBUS
- U1 pad 5: +5V -> VBUS
- U3 pad 1: Net-(U3-Pad1) -> +3V3
Routing:
- net chgsense: track 2.11 -> 40.7 mm, vias 1 -> 2
- net VBUS: track 0.00 -> 25.6 mm
- net +5V: track 2647.0 -> 2625.1 mm
- net +3V3: track 472.8 -> 481.3 mm
- net SPI_RES: track 23.1 -> 15.5 mm
- net Earth: track 13.9 -> 7.90 mm, vias 11 -> 10
- net SPI_CS: track 13.8 -> 9.25 mm
- net SPI_IRQ: track 20.4 -> 16.8 mm
- net I2C_SCL: track 31.5 -> 34.7 mm
- net COL07: track 275.1 -> 272.5 mm
- net SPI_SCK: track 13.1 -> 10.7 mm
- net I2C_SDA: track 37.5 -> 39.7 mm
- net ROW02: track 375.6 -> 373.9 mm
- net SPI_MISO: track 12.7 -> 11.2 mm
- net COL12: track 197.8 -> 199.1 mm
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Other:
- rule trace_min: 0.127 -> 0
- board text added: "1.25u"
- board text added: "1.5u"
- board text added: "1u"
- board text added: "1u 7u stab"
- board text added: "2.25u"
- board text added: "6u"
- board text added: "6u 7u"
- board text added: "6u flipped"
- board text added: "6u/7u"
- board text added: "ANSI"
- board text added: "BOOT"
- board text added: "E80-1800 github.com/ebastler/E80-1800 mpwr.xyz"
- board text added: "ISO"
- board text added: "REG"
- board text added: "RST"
- board text added: "STP"

Commit message: improved mounting holes
Parts:
- added H5: MountingHole, MountingHole:MountingHole_4mm, F.Cu at (49.4, 123.8)
- added JP2: RST, Connector_PinHeader_2.54mm:PinHeader_1x02_P2.54mm_Vertical, B.Cu at (80.1, 111.9)
- added JP3: BOOT, Connector_PinHeader_2.54mm:PinHeader_1x02_P2.54mm_Vertical, B.Cu at (80.1, 116.5)
- J4: value Conn_01x05 -> BATT
- moved J3 0.12 mm to (316.2, -26.9)
- renumbered D2007 to D10, D2008 to D11, D2009 to D12, D2010 to D13, D2011 to D14, D2012 to D15, D2013 to D16, D2014 to D17, D2015 to D18, D2016 to D19, D2017 to D20, D2018 to D21, D2019 to D22, D2020 to D23, D2021 to D24, D2022 to D25, D2023 to D26, D2024 to D27, D2025 to D28, D2026 to D29, D2027 to D30, D2028 to D31, D2029 to D32, D2030 to D33, D2031 to D34, D2032 to D35, D2033 to D36, D2034 to D37, D2035 to D38, D2036 to D39, D2001 to D4, D2037 to D40, D2038 to D41, D2039 to D42, D2040 to D43, D2041 to D44, D2042 to D45, D2043 to D46, D2044 to D47, D2045 to D48, D2046 to D49, D2002 to D5, D2047 to D50, D2048 to D51, D2049 to D52, D2050 to D53, D2051 to D54, D2052 to D55, D2053 to D56, D2054 to D57, D2003 to D6, D2004 to D7, D2005 to D8, D2006 to D9, H3001 to H4, MX2001 to MX1, MX2010 to MX10, MX2100 to MX100, MX2101 to MX101, MX2102 to MX102, MX2103 to MX103, MX2104 to MX104, MX2105 to MX105, MX2106 to MX106, MX2107 to MX107, MX2108 to MX108, MX2109 to MX109, MX2011 to MX11, MX2110 to MX110, MX2111 to MX111, MX2112 to MX112, MX2113 to MX113, MX2114 to MX114, MX2115 to MX115, MX2012 to MX12, MX2013 to MX13, MX2014 to MX14, MX2015 to MX15, MX2016 to MX16, MX2017 to MX17, MX2018 to MX18, MX2019 to MX19, MX2002 to MX2, MX2020 to MX20, MX2021 to MX21, MX2022 to MX22, MX2023 to MX23, MX2024 to MX24, MX2025 to MX25, MX2026 to MX26, MX2027 to MX27, MX2028 to MX28, MX2029 to MX29, MX2003 to MX3, MX2030 to MX30, MX2031 to MX31, MX2032 to MX32, MX2033 to MX33, MX2034 to MX34, MX2035 to MX35, MX2036 to MX36, MX2037 to MX37, MX2038 to MX38, MX2039 to MX39, MX2004 to MX4, MX2040 to MX40, MX2041 to MX41, MX2042 to MX42, MX2043 to MX43, MX2044 to MX44, MX2045 to MX45, MX2046 to MX46, MX2047 to MX47, MX2048 to MX48, MX2049 to MX49, MX2005 to MX5, MX2050 to MX50, MX2051 to MX51, MX2052 to MX52, MX2053 to MX53, MX2054 to MX54, MX2055 to MX55, MX2056 to MX56, MX2057 to MX57, MX2058 to MX58, MX2059 to MX59, MX2006 to MX6, MX2060 to MX60, MX2061 to MX61, MX2062 to MX62, MX2063 to MX63, MX2064 to MX64, MX2065 to MX65, MX2066 to MX66, MX2067 to MX67, MX2068 to MX68, MX2069 to MX69, MX2007 to MX7, MX2070 to MX70, MX2071 to MX71, MX2072 to MX72, MX2073 to MX73, MX2074 to MX74, MX2075 to MX75, MX2076 to MX76, MX2077 to MX77, MX2078 to MX78, MX2079 to MX79, MX2008 to MX8, MX2080 to MX80, MX2081 to MX81, MX2082 to MX82, MX2083 to MX83, MX2084 to MX84, MX2085 to MX85, MX2086 to MX86, MX2087 to MX87, MX2088 to MX88, MX2089 to MX89, MX2009 to MX9, MX2090 to MX90, MX2091 to MX91, MX2092 to MX92, MX2093 to MX93, MX2094 to MX94, MX2095 to MX95, MX2096 to MX96, MX2097 to MX97, MX2098 to MX98, MX2099 to MX99, R2086 to R100, R2087 to R101, R2088 to R102, R2089 to R103, R2090 to R104, R2091 to R105, R2092 to R106, R2093 to R107, R2094 to R108, R2095 to R109, R2096 to R110, R2097 to R111, R2098 to R112, R2099 to R113, R2100 to R114, R2101 to R115, R2102 to R116, R2103 to R117, R2104 to R118, R2105 to R119, R2106 to R120, R2107 to R121, R2001 to R15, R2002 to R16, R2003 to R17, R2004 to R18, R2005 to R19, R2006 to R20, R2007 to R21, R2008 to R22, R2009 to R23, R2010 to R24, R2011 to R25, R2012 to R26, R2013 to R27, R2014 to R28, R2015 to R29, R2016 to R30, R2017 to R31, R2018 to R32, R2019 to R33, R2020 to R34, R2021 to R35, R2022 to R36, R2023 to R37, R2024 to R38, R2025 to R39, R2026 to R40, R2027 to R41, R2028 to R42, R2029 to R43, R2030 to R44, R2031 to R45, R2032 to R46, R2033 to R47, R2034 to R48, R2035 to R49, R2036 to R50, R2037 to R51, R2038 to R52, R2039 to R53, R2040 to R54, R2041 to R55, R2042 to R56, R2043 to R57, R2044 to R58, R2045 to R59, R2046 to R60, R2047 to R61, R2048 to R62, R2049 to R63, R2050 to R64, R2051 to R65, R2052 to R66, R2053 to R67, R2054 to R68, R2055 to R69, R2056 to R70, R2057 to R71, R2058 to R72, R2059 to R73, R2060 to R74, R2061 to R75, R2062 to R76, R2063 to R77, R2064 to R78, R2065 to R79, R2066 to R80, R2067 to R81, R2068 to R82, R2069 to R83, R2070 to R84, R2071 to R85, R2072 to R86, R2073 to R87, R2074 to R88, R2075 to R89, R2076 to R90, R2077 to R91, R2078 to R92, R2079 to R93, R2080 to R94, R2081 to R95, R2082 to R96, R2083 to R97, R2084 to R98, R2085 to R99
Connections:
- J1 pad MP: (no net) -> GND
- J4 pad MP: (no net) -> GND
Routing:
- net /BOOT: track 369.0 -> 379.6 mm
- net /RST: track 338.3 -> 348.8 mm
- net +3V3: track 481.3 -> 488.3 mm
- net Net-(D52-Pad1): track 68.1 -> 72.0 mm
- net +5V: track 2625.1 -> 2626.1 mm
Other:
- outline, holes or cut-outs redrawn
- board text added: "3V3"
- board text added: "GND"
- board text added: "I²C"
- board text added: "SCL"
- board text added: "SDA"

Commit message: minor routing changes
Parts:
- added C1: 10uF, kicad-keyboard-parts:CP_EIA-3216-18_Kemet-A_stealth, B.Cu at (275.5, -24.5)
- C10: renamed from C9; footprint Capacitor_SMD:C_0603_1608Metric_Pad1.05x0.95mm_HandSolder -> kicad-keyboard-parts:C_0603_1608Metric_stealth
- C11: renamed from C10; footprint Capacitor_SMD:C_0603_1608Metric_Pad1.05x0.95mm_HandSolder -> kicad-keyboard-parts:C_0603_1608Metric_stealth
- C12: renamed from C11; footprint Capacitor_SMD:C_0603_1608Metric_Pad1.05x0.95mm_HandSolder -> kicad-keyboard-parts:C_0603_1608Metric_stealth
- C13: renamed from C12; footprint Capacitor_SMD:C_0603_1608Metric_Pad1.05x0.95mm_HandSolder -> kicad-keyboard-parts:C_0603_1608Metric_stealth
- C14: renamed from C13; footprint Capacitor_SMD:C_0603_1608Metric_Pad1.05x0.95mm_HandSolder -> kicad-keyboard-parts:C_0603_1608Metric_stealth
- C15: renamed from C14; footprint Capacitor_SMD:C_0603_1608Metric_Pad1.05x0.95mm_HandSolder -> kicad-keyboard-parts:C_0603_1608Metric_stealth
- C16: renamed from C15; footprint Capacitor_SMD:C_0603_1608Metric_Pad1.05x0.95mm_HandSolder -> kicad-keyboard-parts:C_0603_1608Metric_stealth
- C2: renamed from C1; footprint Capacitor_Tantalum_SMD:CP_EIA-3216-18_Kemet-A -> kicad-keyboard-parts:CP_EIA-3216-18_Kemet-A_stealth
- C3: renamed from C2; footprint Capacitor_SMD:C_0603_1608Metric_Pad1.05x0.95mm_HandSolder -> kicad-keyboard-parts:C_0603_1608Metric_stealth
- C4: renamed from C3; footprint Capacitor_SMD:C_0603_1608Metric_Pad1.05x0.95mm_HandSolder -> kicad-keyboard-parts:C_0603_1608Metric_stealth
- C5: renamed from C4; footprint Capacitor_SMD:C_0603_1608Metric_Pad1.05x0.95mm_HandSolder -> kicad-keyboard-parts:C_0603_1608Metric_stealth
- C6: renamed from C5; footprint Capacitor_SMD:C_0603_1608Metric_Pad1.05x0.95mm_HandSolder -> kicad-keyboard-parts:C_0603_1608Metric_stealth
- C7: renamed from C6; footprint Capacitor_SMD:C_0603_1608Metric_Pad1.05x0.95mm_HandSolder -> kicad-keyboard-parts:C_0603_1608Metric_stealth
- C8: renamed from C7; footprint Capacitor_SMD:C_0603_1608Metric_Pad1.05x0.95mm_HandSolder -> kicad-keyboard-parts:C_0603_1608Metric_stealth
- C9: renamed from C8; footprint Capacitor_SMD:C_0603_1608Metric_Pad1.05x0.95mm_HandSolder -> kicad-keyboard-parts:C_0603_1608Metric_stealth
- D10, D11, D12, D13, D14, D15, D16, D17, D18, D19, D20, D21, D22, D23, D24, D25, D26, D27, D28, D29, D30, D31, D32, D33, D34, D35, D36, D37, D38, D39, D4, D40, D41, D42, D43, D44, D45, D46, D47, D48, D49, D5, D50, D51, D52, D53, D54, D55, D56, D57, D6, D7, D8, D9, Q1, U2: footprint Package_TO_SOT_SMD:SOT-23 -> kicad-keyboard-parts:SOT-23_stealth
- R1, R10, R100, R101, R102, R103, R104, R105, R106, R107, R108, R109, R11, R110, R111, R112, R113, R114, R115, R116, R117, R118, R119, R12, R120, R121, R13, R14, R15, R16, R17, R18, R19, R2, R20, R21, R22, R23, R24, R25, R26, R27, R28, R29, R3, R30, R31, R32, R33, R34, R35, R36, R37, R38, R39, R4, R40, R41, R42, R43, R44, R45, R46, R47, R48, R49, R5, R50, R51, R52, R53, R54, R55, R56, R57, R58, R59, R6, R60, R61, R62, R63, R64, R65, R66, R67, R68, R69, R7, R70, R71, R72, R73, R74, R75, R76, R77, R78, R79, R8, R80, R81, R82, R83, R84, R85, R86, R87, R88, R89, R9, R90, R91, R92, R93, R94, R95, R96, R97, R98, R99: footprint Resistor_SMD:R_0603_1608Metric_Pad1.05x0.95mm_HandSolder -> kicad-keyboard-parts:R_0603_1608Metric_stealth
- SW1, SW2: footprint random-keyboard-parts:SKQG-1155865 -> Button_Switch_SMD:SW_SPST_SKQG_WithoutStem
- moved C4 1.03 mm to (269.1, -24.2)
- moved C3 0.65 mm to (269.1, -22.3)
- moved JP2 0.10 mm to (80.1, 112.0)
- turned SW1 to 180 degrees
- turned SW2 to 180 degrees
Routing:
- net GND: track 7.54 -> 10.2 mm, vias 107 -> 109
- net +3V3: track 488.3 -> 487.1 mm
- net /RST: track 348.8 -> 349.8 mm
- net /BOOT: track 379.6 -> 378.7 mm
- net COL09: track 286.1 -> 287.0 mm
- net SPI_IRQ: track 16.8 -> 17.5 mm
- net COL10: track 234.6 -> 235.1 mm
Other:
- board text added: "RES"
- board text added: "USB"
