File: E80-1800-pcb-universal/E80-1800-Matrix.kicad_sch (KiCad schematic)
At the start: 276 parts

Commit message: updated to v1.2 (switch to marbastlib)
Parts:
- added D100, D101, D102, D103, D104, D105, D106, D107, D108, D109, D110, D111, D112, D113, D114, D115, D116, D118, D119, D120, D121, D122, D123, D124, D125, D126, D127, D128, D129, D130, D131, D132, D133, D134, D135, D136, D137, D138, D139, D140, D141, D142, D143, D144, D145, D146, D147, D148, D149, D150, D151, D152, D153, D154, D155, D157, D158, D160, D161, D162, D163, D165, D166, D168, D169, D170, D171, D172, D59, D60, D61, D62, D63, D64, D65, D66, D67, D68, D69, D70, D71, D72, D73, D74, D75, D76, D77, D78, D79, D80, D81, D82, D83, D84, D85, D86, D87, D88, D89, D90, D91, D92, D93, D94, D95, D96, D97, D98, D99: 3mm, marbastlib-mx:LED_MX_3mm, symbol Device:LED_Small
- added D117, D156, D159, D164, D167: 3mm, marbastlib-mx:LED_MX_3mm-FLIPPED, symbol Device:LED_Small
- added S1: lshift, marbastlib-mx:STAB_MX_2.25u, symbol marbastlib-mx:MX_stab
- added S2: 6u, marbastlib-mx:STAB_MX_6u, symbol marbastlib-mx:MX_stab
- added S3: 7u, marbastlib-mx:STAB_MX_7u, symbol marbastlib-mx:MX_stab
- added S4: ansi_ent, marbastlib-mx:STAB_MX_2.25u, symbol marbastlib-mx:MX_stab
- added S5: iso_ent, marbastlib-mx:STAB_MX_ISO_FLIPPED, symbol marbastlib-mx:MX_stab
- added S6: backspace, marbastlib-mx:STAB_MX_2u, symbol marbastlib-mx:MX_stab
- added S7: np_ent, marbastlib-mx:STAB_MX_2u, symbol marbastlib-mx:MX_stab
- MX1, MX10, MX11, MX12, MX13, MX14, MX15, MX16, MX17, MX18, MX19, MX2, MX20, MX21, MX22, MX23, MX24, MX25, MX26, MX27, MX28, MX29, MX3, MX30, MX31, MX32, MX33, MX34, MX36, MX37, MX38, MX39, MX4, MX41, MX42, MX43, MX44, MX45, MX46, MX47, MX48, MX49, MX5, MX50, MX51, MX52, MX54, MX55, MX56, MX57, MX6, MX60, MX61, MX62, MX63, MX64, MX65, MX66, MX67, MX68, MX69, MX7, MX70, MX71, MX74, MX75, MX76, MX8, MX80, MX81, MX82, MX83, MX84, MX85, MX86, MX87, MX88, MX89, MX9, MX90, MX92, MX93, MX94, MX95: value MX-LED -> MX_SW_solder; footprint MX_Only:MXOnly-1U -> marbastlib-mx:SW_MX_1u; symbol MX_Alps_Hybrid:MX-LED -> marbastlib-mx:MX_SW_solder
- MX100: renamed from MX99; value alt_1u -> MX_SW_solder; footprint MX_Only:MXOnly-1U-FLIPPED -> marbastlib-mx:SW_MX_1u; symbol MX_Alps_Hybrid:MX-LED -> marbastlib-mx:MX_SW_solder
- MX101: renamed from MX111; value alt_1.5u -> MX_SW_solder; footprint MX_Only:MXOnly-1.5U -> marbastlib-mx:SW_MX_1u; symbol MX_Alps_Hybrid:MX-LED -> marbastlib-mx:MX_SW_solder
- MX102: renamed from MX100; value space_6u -> MX_SW_solder; footprint MX_Only:MXOnly-6U -> marbastlib-mx:SW_MX_1u; symbol MX_Alps_Hybrid:MX-LED -> marbastlib-mx:MX_SW_solder
- MX103: renamed from MX112; value space_7u -> MX_SW_solder; footprint MX_Only:MXOnly-7U -> marbastlib-mx:SW_MX_1u; symbol MX_Alps_Hybrid:MX-LED -> marbastlib-mx:MX_SW_solder
- MX104: renamed from MX115; value space_6u_flipped -> MX_SW_solder; footprint MX_Only:MXOnly-1U -> marbastlib-mx:SW_MX_1u; symbol MX_Alps_Hybrid:MX-LED -> marbastlib-mx:MX_SW_solder
- MX105: renamed from MX101; value ralt_1u -> MX_SW_solder; footprint MX_Only:MXOnly-1U -> marbastlib-mx:SW_MX_1u; symbol MX_Alps_Hybrid:MX-LED -> marbastlib-mx:MX_SW_solder
- MX106: renamed from MX113; value ralt_1.5u -> MX_SW_solder; footprint MX_Only:MXOnly-1.5U-FLIPPED -> marbastlib-mx:SW_MX_1u; symbol MX_Alps_Hybrid:MX-LED -> marbastlib-mx:MX_SW_solder
- MX107: renamed from MX102; value rsuper_1u -> MX_SW_solder; footprint MX_Only:MXOnly-1U -> marbastlib-mx:SW_MX_1u; symbol MX_Alps_Hybrid:MX-LED -> marbastlib-mx:MX_SW_solder
- MX108: renamed from MX103; value menu_1u -> MX_SW_solder; footprint MX_Only:MXOnly-1U -> marbastlib-mx:SW_MX_1u; symbol MX_Alps_Hybrid:MX-LED -> marbastlib-mx:MX_SW_solder
- MX109: renamed from MX104; value rctrl_1u -> MX_SW_solder; footprint MX_Only:MXOnly-1U-FLIPPED -> marbastlib-mx:SW_MX_1u; symbol MX_Alps_Hybrid:MX-LED -> marbastlib-mx:MX_SW_solder
- MX110: renamed from MX114; value rctrl_1.5u -> MX_SW_solder; footprint MX_Only:MXOnly-1.5U -> marbastlib-mx:SW_MX_1u; symbol MX_Alps_Hybrid:MX-LED -> marbastlib-mx:MX_SW_solder
- MX111: renamed from MX105; value MX-LED -> MX_SW_solder; footprint MX_Only:MXOnly-1U -> marbastlib-mx:SW_MX_1u; symbol MX_Alps_Hybrid:MX-LED -> marbastlib-mx:MX_SW_solder
- MX112: renamed from MX106; value MX-LED -> MX_SW_solder; footprint MX_Only:MXOnly-1U -> marbastlib-mx:SW_MX_1u; symbol MX_Alps_Hybrid:MX-LED -> marbastlib-mx:MX_SW_solder
- MX113: renamed from MX107; value MX-LED -> MX_SW_solder; footprint MX_Only:MXOnly-1U -> marbastlib-mx:SW_MX_1u; symbol MX_Alps_Hybrid:MX-LED -> marbastlib-mx:MX_SW_solder
- MX114: renamed from MX108; value MX-LED -> MX_SW_solder; footprint MX_Only:MXOnly-1U -> marbastlib-mx:SW_MX_1u; symbol MX_Alps_Hybrid:MX-LED -> marbastlib-mx:MX_SW_solder
- MX115: renamed from MX109; value MX-LED -> MX_SW_solder; footprint MX_Only:MXOnly-1U -> marbastlib-mx:SW_MX_1u; symbol MX_Alps_Hybrid:MX-LED -> marbastlib-mx:MX_SW_solder
- MX35: value Backspace_2u -> MX_SW_solder; footprint MX_Only:MXOnly-2U -> marbastlib-mx:SW_MX_1u; symbol MX_Alps_Hybrid:MX-LED -> marbastlib-mx:MX_SW_solder
- MX40: value tab -> MX_SW_solder; footprint MX_Only:MXOnly-1.5U -> marbastlib-mx:SW_MX_1u; symbol MX_Alps_Hybrid:MX-LED -> marbastlib-mx:MX_SW_solder
- MX53: value \_ansi -> MX_SW_solder; footprint MX_Only:MXOnly-1.5U -> marbastlib-mx:SW_MX_1u; symbol MX_Alps_Hybrid:MX-LED -> marbastlib-mx:MX_SW_solder
- MX58: value caps -> MX_SW_solder; footprint MX_Only:MXOnly-1.75U-FLIPPED -> marbastlib-mx:SW_MX_1u; symbol MX_Alps_Hybrid:MX-LED -> marbastlib-mx:MX_SW_solder
- MX59: value caps_stepped -> MX_SW_solder; footprint MX_Only:MXOnly-1.25U -> marbastlib-mx:SW_MX_1u; symbol MX_Alps_Hybrid:MX-LED -> marbastlib-mx:MX_SW_solder
- MX72: value enter_iso -> MX_SW_solder; footprint MX_Only:MXOnly-ISO-ROTATED-ReversedStabilizers -> marbastlib-mx:SW_MX_1u; symbol MX_Alps_Hybrid:MX-LED -> marbastlib-mx:MX_SW_solder
- MX73: value enter_ansi -> MX_SW_solder; footprint MX_Only:MXOnly-2.25U -> marbastlib-mx:SW_MX_1u; symbol MX_Alps_Hybrid:MX-LED -> marbastlib-mx:MX_SW_solder
- MX77: value + -> MX_SW_solder; footprint MX_Only:MXOnly-1U -> marbastlib-mx:SW_MX_1u; symbol MX_Alps_Hybrid:MX-LED -> marbastlib-mx:MX_SW_solder
- MX78: value lshift_iso -> MX_SW_solder; footprint MX_Only:MXOnly-1.25U -> marbastlib-mx:SW_MX_1u; symbol MX_Alps_Hybrid:MX-LED -> marbastlib-mx:MX_SW_solder
- MX79: value lshift_ansi -> MX_SW_solder; footprint MX_Only:MXOnly-2.25U -> marbastlib-mx:SW_MX_1u; symbol MX_Alps_Hybrid:MX-LED -> marbastlib-mx:MX_SW_solder
- MX91: value rshift -> MX_SW_solder; footprint MX_Only:MXOnly-1.75U -> marbastlib-mx:SW_MX_1u; symbol MX_Alps_Hybrid:MX-LED -> marbastlib-mx:MX_SW_solder
- MX96: value enter_numpad -> MX_SW_solder; footprint MX_Only:MXOnly-ISO -> marbastlib-mx:SW_MX_1u; symbol MX_Alps_Hybrid:MX-LED -> marbastlib-mx:MX_SW_solder
- MX97: value ctrl_1u -> MX_SW_solder; footprint MX_Only:MXOnly-1U -> marbastlib-mx:SW_MX_1u; symbol MX_Alps_Hybrid:MX-LED -> marbastlib-mx:MX_SW_solder
- MX98: renamed from MX110; value ctrl_1.5u -> MX_SW_solder; footprint MX_Only:MXOnly-1.5U-FLIPPED -> marbastlib-mx:SW_MX_1u; symbol MX_Alps_Hybrid:MX-LED -> marbastlib-mx:MX_SW_solder
- MX99: renamed from MX98; value super_1u -> MX_SW_solder; footprint MX_Only:MXOnly-1U -> marbastlib-mx:SW_MX_1u; symbol MX_Alps_Hybrid:MX-LED -> marbastlib-mx:MX_SW_solder
- renumbered R120 to R111, R121 to R112, R111 to R113, R112 to R114, R113 to R115, R114 to R116, R115 to R117, R116 to R118, R117 to R119, R118 to R120, R119 to R121
Connections:
- net +5V: now also D100.2 (A), D101.2 (A), D102.2 (A), D103.2 (A), D104.2 (A), D105.2 (A), D106.2 (A), D107.2 (A), D108.2 (A), D109.2 (A), D110.2 (A), D111.2 (A), D112.2 (A), D113.2 (A), D114.2 (A), D115.2 (A), D116.2 (A), D117.2 (A), D118.2 (A), D119.2 (A), D120.2 (A), D121.2 (A), D122.2 (A), D123.2 (A), D124.2 (A), D125.2 (A), D126.2 (A), D127.2 (A), D128.2 (A), D129.2 (A), D130.2 (A), D131.2 (A), D132.2 (A), D133.2 (A), D134.2 (A), D135.2 (A), D136.2 (A), D137.2 (A), D138.2 (A), D139.2 (A), D140.2 (A), D141.2 (A), D142.2 (A), D143.2 (A), D144.2 (A), D145.2 (A), D146.2 (A), D147.2 (A), D148.2 (A), D149.2 (A), D150.2 (A), D151.2 (A), D152.2 (A), D153.2 (A), D154.2 (A), D155.2 (A), D156.2 (A), D157.2 (A), D158.2 (A), D159.2 (A), D160.2 (A), D161.2 (A), D162.2 (A), D163.2 (A), D164.2 (A), D165.2 (A), D166.2 (A), D167.2 (A), D168.2 (A), D169.2 (A), D170.2 (A), D171.2 (A), D172.2 (A), D59.2 (A), D60.2 (A), D61.2 (A), D62.2 (A), D63.2 (A), D64.2 (A), D65.2 (A), D66.2 (A), D67.2 (A), D68.2 (A), D69.2 (A), D70.2 (A), D71.2 (A), D72.2 (A), D73.2 (A), D74.2 (A), D75.2 (A), D76.2 (A), D77.2 (A), D78.2 (A), D79.2 (A), D80.2 (A), D81.2 (A), D82.2 (A), D83.2 (A), D84.2 (A), D85.2 (A), D86.2 (A), D87.2 (A), D88.2 (A), D89.2 (A), D90.2 (A), D91.2 (A), D92.2 (A), D93.2 (A), D94.2 (A), D95.2 (A), D96.2 (A), D97.2 (A), D98.2 (A), D99.2 (A); no longer MX1.3 (LED), MX10.3 (LED), MX100.3 (LED), MX101.3 (LED), MX102.3 (LED), MX103.3 (LED), MX104.3 (LED), MX105.3 (LED), MX106.3 (LED), MX107.3 (LED), MX108.3 (LED), MX109.3 (LED), MX11.3 (LED), MX110.3 (LED), MX111.3 (LED), MX112.3 (LED), MX113.3 (LED), MX114.3 (LED), MX115.3 (LED), MX12.3 (LED), MX13.3 (LED), MX14.3 (LED), MX15.3 (LED), MX16.3 (LED), MX17.3 (LED), MX18.3 (LED), MX19.3 (LED), MX2.3 (LED), MX20.3 (LED), MX21.3 (LED), MX22.3 (LED), MX23.3 (LED), MX24.3 (LED), MX25.3 (LED), MX26.3 (LED), MX27.3 (LED), MX28.3 (LED), MX29.3 (LED), MX3.3 (LED), MX30.3 (LED), MX31.3 (LED), MX32.3 (LED), MX33.3 (LED), MX34.3 (LED), MX35.3 (LED), MX36.3 (LED), MX37.3 (LED), MX38.3 (LED), MX39.3 (LED), MX4.3 (LED), MX40.3 (LED), MX41.3 (LED), MX42.3 (LED), MX43.3 (LED), MX44.3 (LED), MX45.3 (LED), MX46.3 (LED), MX47.3 (LED), MX48.3 (LED), MX49.3 (LED), MX5.3 (LED), MX50.3 (LED), MX51.3 (LED), MX52.3 (LED), MX53.3 (LED), MX54.3 (LED), MX55.3 (LED), MX56.3 (LED), MX57.3 (LED), MX58.3 (LED), MX59.3 (LED), MX6.3 (LED), MX60.3 (LED), MX61.3 (LED), MX62.3 (LED), MX63.3 (LED), MX64.3 (LED), MX65.3 (LED), MX66.3 (LED), MX67.3 (LED), MX68.3 (LED), MX69.3 (LED), MX7.3 (LED), MX70.3 (LED), MX71.3 (LED), MX72.3 (LED), MX73.3 (LED), MX74.3 (LED), MX75.3 (LED), MX76.3 (LED), MX77.3 (LED), MX78.3 (LED), MX79.3 (LED), MX8.3 (LED), MX80.3 (LED), MX81.3 (LED), MX82.3 (LED), MX83.3 (LED), MX84.3 (LED), MX85.3 (LED), MX86.3 (LED), MX87.3 (LED), MX88.3 (LED), MX89.3 (LED), MX9.3 (LED), MX90.3 (LED), MX91.3 (LED), MX92.3 (LED), MX93.3 (LED), MX94.3 (LED), MX95.3 (LED), MX96.3 (LED), MX97.3 (LED), MX98.3 (LED), MX99.3 (LED)
- net at R15.2: now also D59.1 (K); no longer MX1.4 (LEDGND)
- net at R16.2: now also D60.1 (K); no longer MX2.4 (LEDGND)
- net at R17.2: now also D61.1 (K); no longer MX3.4 (LEDGND)
- net at R18.2: now also D62.1 (K); no longer MX4.4 (LEDGND)
- net at R19.2: now also D63.1 (K); no longer MX5.4 (LEDGND)
- net at R20.2: now also D64.1 (K); no longer MX6.4 (LEDGND)
- net at R21.2: now also D65.1 (K); no longer MX7.4 (LEDGND)
- net at R22.2: now also D66.1 (K); no longer MX8.4 (LEDGND)
- net at R23.2: now also D67.1 (K); no longer MX9.4 (LEDGND)
- net at R24.2: now also D68.1 (K); no longer MX10.4 (LEDGND)
- net at R25.2: now also D69.1 (K); no longer MX11.4 (LEDGND)
- net at R26.2: now also D70.1 (K); no longer MX12.4 (LEDGND)
- net at R27.2: now also D71.1 (K); no longer MX13.4 (LEDGND)
- net at R28.2: now also D72.1 (K); no longer MX14.4 (LEDGND)
- net at R29.2: now also D73.1 (K); no longer MX15.4 (LEDGND)
- net at R30.2: now also D74.1 (K); no longer MX16.4 (LEDGND)
- net at R31.2: now also D75.1 (K); no longer MX17.4 (LEDGND)
- net at R36.2: now also D80.1 (K); no longer MX22.4 (LEDGND)
- net at R37.2: now also D81.1 (K); no longer MX23.4 (LEDGND)
- net at R38.2: now also D82.1 (K); no longer MX24.4 (LEDGND)
- net at R39.2: now also D83.1 (K); no longer MX25.4 (LEDGND)
- net at R40.2: now also D84.1 (K); no longer MX26.4 (LEDGND)
- net at R41.2: now also D85.1 (K); no longer MX27.4 (LEDGND)
- net at R42.2: now also D86.1 (K); no longer MX28.4 (LEDGND)
- net at R43.2: now also D87.1 (K); no longer MX29.4 (LEDGND)
- net at R44.2: now also D88.1 (K); no longer MX30.4 (LEDGND)
- net at R45.2: now also D89.1 (K); no longer MX31.4 (LEDGND)
- net at R46.2: now also D90.1 (K); no longer MX32.4 (LEDGND)
- net at R47.2: now also D91.1 (K); no longer MX33.4 (LEDGND)
- net at R48.2: now also D92.1 (K); no longer MX34.4 (LEDGND)
- net at R49.2: now also D93.1 (K); no longer MX35.4 (LEDGND)
- net at R50.2: now also D94.1 (K); no longer MX36.4 (LEDGND)
- net at R51.2: now also D95.1 (K); no longer MX37.4 (LEDGND)
- net at R52.2: now also D96.1 (K); no longer MX38.4 (LEDGND)
- net at R53.2: now also D97.1 (K); no longer MX39.4 (LEDGND)
- net at R112.2: now also D161.1 (K); no longer MX104.4 (LEDGND)
- net at R71.2: now also D115.1 (K); no longer MX57.4 (LEDGND)
- net at R70.2: now also D114.1 (K); no longer MX56.4 (LEDGND)
- net at R69.2: now also D113.1 (K); no longer MX55.4 (LEDGND)
- net at R68.2: now also D112.1 (K); no longer MX54.4 (LEDGND)
- net at R66.2: now also D110.1 (K); no longer MX52.4 (LEDGND)
- net at R65.2: now also D109.1 (K); no longer MX51.4 (LEDGND)
- net at R64.2: now also D108.1 (K); no longer MX50.4 (LEDGND)
- net at R63.2: now also D107.1 (K); no longer MX49.4 (LEDGND)
- net at R62.2: now also D106.1 (K); no longer MX48.4 (LEDGND)
- net at R61.2: now also D105.1 (K); no longer MX47.4 (LEDGND)
- net at R60.2: now also D104.1 (K); no longer MX46.4 (LEDGND)
- net at R59.2: now also D103.1 (K); no longer MX45.4 (LEDGND)
- net at R58.2: now also D102.1 (K); no longer MX44.4 (LEDGND)
- net at R57.2: now also D101.1 (K); no longer MX43.4 (LEDGND)
- net at R56.2: now also D100.1 (K); no longer MX42.4 (LEDGND)
- net at R55.2: now also D99.1 (K); no longer MX41.4 (LEDGND)
- net at R54.2: now also D98.1 (K); no longer MX40.4 (LEDGND)
- net at R89.2: now also D135.1 (K); no longer MX77.4 (LEDGND)
- net at R88.2: now also D134.1 (K); no longer MX76.4 (LEDGND)
- net at R87.2: now also D133.1 (K); no longer MX75.4 (LEDGND)
- net at R86.2: now also D132.1 (K); no longer MX74.4 (LEDGND)
- net at R84.2: now also D129.1 (K); no longer MX71.4 (LEDGND)
- net at R83.2: now also D128.1 (K); no longer MX70.4 (LEDGND)
- net at R82.2: now also D127.1 (K); no longer MX69.4 (LEDGND)
- net at R81.2: now also D126.1 (K); no longer MX68.4 (LEDGND)
- net at R80.2: now also D125.1 (K); no longer MX67.4 (LEDGND)
- net at R79.2: now also D124.1 (K); no longer MX66.4 (LEDGND)
- net at R78.2: now also D123.1 (K); no longer MX65.4 (LEDGND)
- net at R77.2: now also D122.1 (K); no longer MX64.4 (LEDGND)
- net at R76.2: now also D121.1 (K); no longer MX63.4 (LEDGND)
- net at R75.2: now also D120.1 (K); no longer MX62.4 (LEDGND)
- net at R74.2: now also D119.1 (K); no longer MX61.4 (LEDGND)
- net at R73.2: now also D118.1 (K); no longer MX60.4 (LEDGND)
- net at R107.2: now also D154.1 (K); no longer MX96.4 (LEDGND)
- net at R106.2: now also D153.1 (K); no longer MX95.4 (LEDGND)
- net at R105.2: now also D152.1 (K); no longer MX94.4 (LEDGND)
- net at R104.2: now also D151.1 (K); no longer MX93.4 (LEDGND)
- net at R103.2: now also D150.1 (K); no longer MX92.4 (LEDGND)
- net at R102.2: now also D149.1 (K); no longer MX91.4 (LEDGND)
- net at R101.2: now also D148.1 (K); no longer MX90.4 (LEDGND)
- net at R100.2: now also D147.1 (K); no longer MX89.4 (LEDGND)
- net at R99.2: now also D146.1 (K); no longer MX88.4 (LEDGND)
- net at R98.2: now also D145.1 (K); no longer MX87.4 (LEDGND)
- net at R97.2: now also D144.1 (K); no longer MX86.4 (LEDGND)
- net at R96.2: now also D143.1 (K); no longer MX85.4 (LEDGND)
- net at R95.2: now also D142.1 (K); no longer MX84.4 (LEDGND)
- net at R94.2: now also D141.1 (K); no longer MX83.4 (LEDGND)
- net at R93.2: now also D140.1 (K); no longer MX82.4 (LEDGND)
- net at R92.2: now also D139.1 (K); no longer MX81.4 (LEDGND)
- net at R91.2: now also D138.1 (K); no longer MX80.4 (LEDGND)
- net at R121.2: now also D172.1 (K); no longer MX115.4 (LEDGND)
- net at R120.2: now also D171.1 (K); no longer MX114.4 (LEDGND)
- net at R119.2: now also D170.1 (K); no longer MX113.4 (LEDGND)
- net at R118.2: now also D169.1 (K); no longer MX112.4 (LEDGND)
- net at R117.2: now also D168.1 (K); no longer MX111.4 (LEDGND)
- net at R115.2: now also D165.1 (K); no longer MX108.4 (LEDGND)
- net at R113.2: now also D162.1 (K); no longer MX105.4 (LEDGND)
- net at R109.2: now also D157.1 (K); no longer MX99.4 (LEDGND)
- net at R67.2: now also D111.1 (K); no longer MX53.4 (LEDGND)
- net at R32.2: now also D76.1 (K); no longer MX18.4 (LEDGND)
- net at R33.2: now also D77.1 (K); no longer MX19.4 (LEDGND)
- net at R34.2: now also D78.1 (K); no longer MX20.4 (LEDGND)
- net at R35.2: now also D79.1 (K); no longer MX21.4 (LEDGND)
- new net: D160.1 (K), R111.2
- new net: D130.1 (K), D131.1 (K), R85.2
- new net: D116.1 (K), D117.1 (K), R72.2
- new net: D136.1 (K), D137.1 (K), R90.2
- new net: D163.1 (K), D164.1 (K), R114.2
- new net: D166.1 (K), D167.1 (K), R116.2
- new net: D158.1 (K), D159.1 (K), R110.2
- new net: D155.1 (K), D156.1 (K), R108.2
Other:
- moved on the sheet: D10, D11, D12, D13, D14, D15, D16, D17, D18, D19, D20, D21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

Commit message: update to PCM marbastlib and KC8
Parts:
- D100, D101, D102, D103, D104, D105, D106, D107, D108, D109, D110, D111, D112, D113, D114, D115, D116, D118, D119, D120, D121, D122, D123, D124, D125, D126, D127, D128, D129, D130, D131, D132, D133, D134, D135, D136, D137, D138, D139, D140, D141, D142, D143, D144, D145, D146, D147, D148, D149, D150, D151, D152, D153, D154, D155, D157, D158, D160, D161, D162, D163, D165, D166, D168, D169, D170, D171, D172, D59, D60, D61, D62, D63, D64, D65, D66, D67, D68, D69, D70, D71, D72, D73, D74, D75, D76, D77, D78, D79, D80, D81, D82, D83, D84, D85, D86, D87, D88, D89, D90, D91, D92, D93, D94, D95, D96, D97, D98, D99: footprint marbastlib-mx:LED_MX_3mm -> PCM_marbastlib-mx:LED_MX_3mm
- D117, D156, D159, D164, D167: footprint marbastlib-mx:LED_MX_3mm-FLIPPED -> PCM_marbastlib-mx:LED_MX_3mm-ROT
- MX1, MX10, MX100, MX101, MX102, MX103, MX104, MX105, MX106, MX107, MX108, MX109, MX11, MX110, MX111, MX112, MX113, MX114, MX115, MX12, MX13, MX14, MX15, MX16, MX17, MX18, MX19, MX2, MX20, MX21, MX22, MX23, MX24, MX25, MX26, MX27, MX28, MX29, MX3, MX30, MX31, MX32, MX33, MX34, MX35, MX36, MX37, MX38, MX39, MX4, MX40, MX41, MX42, MX43, MX44, MX45, MX46, MX47, MX48, MX49, MX5, MX50, MX51, MX52, MX53, MX54, MX55, MX56, MX57, MX58, MX59, MX6, MX60, MX61, MX62, MX63, MX64, MX65, MX66, MX67, MX68, MX69, MX7, MX70, MX71, MX72, MX73, MX74, MX75, MX76, MX77, MX78, MX79, MX8, MX80, MX81, MX82, MX83, MX84, MX85, MX86, MX87, MX88, MX89, MX9, MX90, MX91, MX92, MX93, MX94, MX95, MX96, MX97, MX98, MX99: footprint marbastlib-mx:SW_MX_1u -> PCM_marbastlib-mx:SW_MX_1u
- S1, S4: footprint marbastlib-mx:STAB_MX_2.25u -> PCM_marbastlib-mx:STAB_MX_2.25u
- S2: footprint marbastlib-mx:STAB_MX_6u -> PCM_marbastlib-mx:STAB_MX_6u
- S3: footprint marbastlib-mx:STAB_MX_7u -> PCM_marbastlib-mx:STAB_MX_7u
- S5: footprint marbastlib-mx:STAB_MX_ISO_FLIPPED -> PCM_marbastlib-mx:STAB_MX_ISO-ROT
- S6, S7: footprint marbastlib-mx:STAB_MX_2u -> PCM_marbastlib-mx:STAB_MX_2u

Commit message: updated jlc production files to current stocks, fixed rotations, moved symbols to PCB marbastlib
Parts:
- MX1, MX10, MX100, MX101, MX102, MX103, MX104, MX105, MX106, MX107, MX108, MX109, MX11, MX110, MX111, MX112, MX113, MX114, MX115, MX12, MX13, MX14, MX15, MX16, MX17, MX18, MX19, MX2, MX20, MX21, MX22, MX23, MX24, MX25, MX26, MX27, MX28, MX29, MX3, MX30, MX31, MX32, MX33, MX34, MX35, MX36, MX37, MX38, MX39, MX4, MX40, MX41, MX42, MX43, MX44, MX45, MX46, MX47, MX48, MX49, MX5, MX50, MX51, MX52, MX53, MX54, MX55, MX56, MX57, MX58, MX59, MX6, MX60, MX61, MX62, MX63, MX64, MX65, MX66, MX67, MX68, MX69, MX7, MX70, MX71, MX72, MX73, MX74, MX75, MX76, MX77, MX78, MX79, MX8, MX80, MX81, MX82, MX83, MX84, MX85, MX86, MX87, MX88, MX89, MX9, MX90, MX91, MX92, MX93, MX94, MX95, MX96, MX97, MX98, MX99: symbol marbastlib-mx:MX_SW_solder -> PCM_marbastlib-mx:MX_SW_solder
- S1, S2, S3, S4, S5, S6, S7: symbol marbastlib-mx:MX_stab -> PCM_marbastlib-mx:MX_stab
